File: SympleSensorBoard.sch (EAGLE design)
At the start: 44 parts, among them IC1 STM32F303K8T6, J1 B2B-XH-A_LF__SN_, J10 B3B-XH-A_LF__SN_, J11 B3B-XH-A_LF__SN_, J12 B4B-XH-A_LF__SN_, J13 B4B-XH-A_LF__SN_, J14 B4B-XH-A_LF__SN_, J15 B4B-XH-A_LF__SN_, J2 B2B-XH-A_LF__SN_, J3 B2B-XH-A_LF__SN_, J4 B2B-XH-A_LF__SN_, J5 B2B-XH-A_LF__SN_, J6 B3B-XH-A_LF__SN_, J7 B3B-XH-A_LF__SN_, J8 B3B-XH-A_LF__SN_, J9 B3B-XH-A_LF__SN_, Y1 CSTCE12M0G55-R0

Commit message: 回路図完成しました
Parts:
- added MOSFET1: IRLML6344TRPBFTR, mukuchin_transistor_fet_igbt:IRLML6344TRPBFTR
- added R18: 10k, rcl:R-US_R0603
- added R19: 1k, rcl:R-US_R0603
- added R20: 2k, rcl:R-US_R0603
Connections:
- new net N$11: J12.3, MOSFET1.D, R18.1
- new net N$13: J12.2, R19.1
- net +3.3V: now also J13.1, J14.1, J15.1
- net +5V: now also J12.1, R18.2
- net ECHO: now also MOSFET1.G
- net GND: now also J12.4, J13.4, J14.4, J15.4, MOSFET1.S, R20.1
- net SCL: now also J13.3, J14.3, J15.3
- net SDA: now also J13.2, J14.2, J15.2
- net TRIG: now also R19.2, R20.2
Other:
- moved on the sheet: J12
Changed lines of the file:
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@@
 <part name="R16" library="rcl" library_urn="urn:adsk.eagle:library:334" deviceset="R-US_" device="R0603" package3d_urn="urn:adsk.eagle:package:23555/3" value="1k"/>
 <part name="R17" library="rcl" library_urn="urn:adsk.eagle:library:334" deviceset="R-US_" device="R0603" package3d_urn="urn:adsk.eagle:package:23555/3" value="2k"/>
+<part name="MOSFET1" library="mukuchin_transistor_fet_igbt" deviceset="IRLML6344TRPBFTR" device=""/>
+<part name="R18" library="rcl" library_urn="urn:adsk.eagle:library:334" deviceset="R-US_" device="R0603" package3d_urn="urn:adsk.eagle:package:23555/3" value="10k"/>
+<part name="R19" library="rcl" library_urn="urn:adsk.eagle:library:334" deviceset="R-US_" device="R0603" package3d_urn="urn:adsk.eagle:package:23555/3" value="1k"/>
+<part name="R20" library="rcl" library_urn="urn:adsk.eagle:library:334" deviceset="R-US_" device="R0603" package3d_urn="urn:adsk.eagle:package:23555/3" value="2k"/>
 </parts>
 <sheets>
@@
 <attribute name="VALUE" x="55.51" y="-181.92" size="1.778" layer="96" align="center-left"/>
 </instance>
-<instance part="J12" gate="G$1" x="-86" y="-96" smashed="yes">
-<attribute name="NAME" x="-69.49" y="-88.38" size="1.778" layer="95" align="center-left"/>
-<attribute name="VALUE" x="-69.49" y="-90.92" size="1.778" layer="96" align="center-left"/>
+<instance part="J12" gate="G$1" x="-72" y="-66" smashed="yes">
+<attribute name="NAME" x="-55.49" y="-58.38" size="1.778" layer="95" align="center-left"/>
+<attribute name="VALUE" x="-55.49" y="-60.92" size="1.778" layer="96" align="center-left"/>
 </instance>
 <instance part="J13" gate="G$1" x="-86" y="-122" smashed="yes">
@@
 <attribute name="NAME" x="17.19" y="-193.5014" size="1.778" layer="95"/>
 <attribute name="VALUE" x="17.19" y="-198.302" size="1.778" layer="96"/>
+</instance>
+<instance part="MOSFET1" gate="G$1" x="-86" y="-77" smashed="yes">
+<attribute name="VALUE" x="-97.43" y="-77" size="1.778" layer="96"/>
+<attribute name="NAME" x="-97.43" y="-74.46" size="1.778" layer="95"/>
+</instance>
+<instance part="R18" gate="G$1" x="-91" y="-64" smashed="yes" rot="R180">
+<attribute name="NAME" x="-87.19" y="-65.4986" size="1.778" layer="95" rot="R180"/>
+<attribute name="VALUE" x="-87.19" y="-60.698" size="1.778" layer="96" rot="R180"/>
+</instance>
+<instance part="R19" gate="G$1" x="-77" y="-83" smashed="yes" rot="R270">
+<attribute name="NAME" x="-75.5014" y="-79.19" size="1.778" layer="95" rot="R270"/>
+<attribute name="VALUE" x="-80.302" y="-79.19" size="1.778" layer="96" rot="R270"/>
+</instance>
+<instance part="R20" gate="G$1" x="-87" y="-94" smashed="yes">
+<attribute name="NAME" x="-90.81" y="-92.5014" size="1.778" layer="95"/>
+<attribute name="VALUE" x="-90.81" y="-97.302" size="1.778" layer="96"/>
 </instance>
 </instances>
@@
 </segment>
 <segment>
-<wire x1="-99" y1="-85" x2="-99" y2="-222" width="0.762" layer="92"/>
+<wire x1="-99" y1="-57" x2="-99" y2="-222" width="0.762" layer="92"/>
 </segment>
 </bus>
@@
 <label x="132" y="-168" size="1.778" layer="95"/>
 </segment>
+<segment>
+<pinref part="J13" gate="G$1" pin="1"/>
+<wire x1="-86" y1="-122" x2="-99" y2="-122" width="0.1524" layer="91"/>
+<label x="-106" y="-122" size="1.778" layer="95"/>
+</segment>
+<segment>
+<pinref part="J14" gate="G$1" pin="1"/>
+<wire x1="-86" y1="-150" x2="-99" y2="-150" width="0.1524" layer="91"/>
+<label x="-106" y="-150" size="1.778" layer="95"/>
+</segment>
+<segment>
+<pinref part="J15" gate="G$1" pin="1"/>
+<wire x1="-86" y1="-181" x2="-99" y2="-181" width="0.1524" layer="91"/>
+<label x="-106" y="-181" size="1.778" layer="95"/>
+</segment>
 </net>
 <net name="GND" class="0">
@@
 <wire x1="15.92" y1="-195" x2="15" y2="-195" width="0.1524" layer="91"/>
 </segment>
+<segment>
+<pinref part="MOSFET1" gate="G$1" pin="S"/>
+<wire x1="-83.46" y1="-84.62" x2="-83.46" y2="-85" width="0.1524" layer="91"/>
+<wire x1="-83.46" y1="-85" x2="-99" y2="-85" width="0.1524" layer="91"/>
+<label x="-105" y="-85" size="1.778" layer="95"/>
+</segment>
+<segment>
+<pinref part="J12" gate="G$1" pin="4"/>
+<wire x1="-72" y1="-73.62" x2="-79" y2="-73.62" width="0.1524" layer="91"/>
+<wire x1="-79" y1="-73.62" x2="-79" y2="-68" width="0.1524" layer="91"/>
+<wire x1="-99" y1="-68" x2="-79" y2="-68" width="0.1524" layer="91"/>
+<label x="-105" y="-68" size="1.778" layer="95"/>
+</segment>
+<segment>
+<pinref part="R20" gate="G$1" pin="1"/>
+<wire x1="-92.08" y1="-94" x2="-99" y2="-94" width="0.1524" layer="91"/>
+<label x="-105" y="-94" size="1.778" layer="95"/>
+</segment>
+<segment>
+<pinref part="J13" gate="G$1" pin="4"/>
+<wire x1="-86" y1="-129.62" x2="-99" y2="-129.62" width="0.1524" layer="91"/>
+<wire x1="-99" y1="-129.62" x2="-99" y2="-130" width="0.1524" layer="91"/>
+<label x="-105" y="-130" size="1.778" layer="95"/>
+</segment>
+<segment>
+<pinref part="J14" gate="G$1" pin="4"/>
+<wire x1="-86" y1="-157.62" x2="-86" y2="-158" width="0.1524" layer="91"/>
+<wire x1="-86" y1="-158" x2="-99" y2="-158" width="0.1524" layer="91"/>
+<label x="-105" y="-158" size="1.778" layer="95"/>
+</segment>
+<segment>
+<pinref part="J15" gate="G$1" pin="4"/>
+<wire x1="-86" y1="-188.62" x2="-99" y2="-188.62" width="0.1524" layer="91"/>
+<wire x1="-99" y1="-188.62" x2="-99" y2="-189" width="0.1524" layer="91"/>
+<label x="-105" y="-189" size="1.778" layer="95"/>
+</segment>
 </net>
 <net name="OSC_IN" class="0">
@@
 <label x="54" y="110" size="1.778" layer="95" rot="R90"/>
 </segment>
+<segment>
+<pinref part="J13" gate="G$1" pin="2"/>
+<wire x1="-86" y1="-124.54" x2="-99" y2="-124.54" width="0.1524" layer="91"/>
+<wire x1="-99" y1="-124.54" x2="-99" y2="-125" width="0.1524" layer="91"/>
+<label x="-105" y="-125" size="1.778" layer="95"/>
+</segment>
+<segment>
+<pinref part="J14" gate="G$1" pin="2"/>
+<wire x1="-86" y1="-152.54" x2="-99" y2="-152.54" width="0.1524" layer="91"/>
+<wire x1="-99" y1="-152.54" x2="-99" y2="-153" width="0.1524" layer="91"/>
+<label x="-105" y="-153" size="1.778" layer="95"/>
+</segment>
+<segment>
+<pinref part="J15" gate="G$1" pin="2"/>
+<wire x1="-86" y1="-183.54" x2="-99" y2="-183.54" width="0.1524" layer="91"/>
+<wire x1="-99" y1="-183.54" x2="-99" y2="-184" width="0.1524" layer="91"/>
+<label x="-105" y="-184" size="1.778" layer="95"/>
+</segment>
 </net>
 <net name="SCL" class="0">
@@
 <label x="57" y="110" size="1.778" layer="95" rot="R90"/>
 </segment>
+<segment>
+<pinref part="J13" gate="G$1" pin="3"/>
+<wire x1="-86" y1="-127.08" x2="-99" y2="-127.08" width="0.1524" layer="91"/>
+<wire x1="-99" y1="-127.08" x2="-99" y2="-127" width="0.1524" layer="91"/>
+<label x="-105" y="-127" size="1.778" layer="95"/>
+</segment>
+<segment>
+<pinref part="J14" gate="G$1" pin="3"/>
+<wire x1="-86" y1="-155.08" x2="-99" y2="-155.08" width="0.1524" layer="91"/>
+<wire x1="-99" y1="-155.08" x2="-99" y2="-155" width="0.1524" layer="91"/>
+<label x="-105" y="-155" size="1.778" layer="95"/>
+</segment>
+<segment>
+<pinref part="J15" gate="G$1" pin="3"/>
+<wire x1="-86" y1="-186.08" x2="-99" y2="-186.08" width="0.1524" layer="91"/>
+<wire x1="-99" y1="-186.08" x2="-99" y2="-186" width="0.1524" layer="91"/>
+<label x="-105" y="-186" size="1.778" layer="95"/>
+</segment>
 </net>
 <net name="ECHO" class="0">
@@
 <label x="59" y="110" size="1.778" layer="95" rot="R90"/>
 </segment>
+<segment>
+<pinref part="MOSFET1" gate="G$1" pin="G"/>
+<wire x1="-91.08" y1="-79.54" x2="-99" y2="-79.54" width="0.1524" layer="91"/>
+<wire x1="-99" y1="-79.54" x2="-99" y2="-80" width="0.1524" layer="91"/>
+<label x="-107" y="-80" size="1.778" layer="95"/>
+</segment>
 </net>
 <net name="TRIG" class="0">
@@
 <wire x1="61.86" y1="109" x2="62" y2="109" width="0.1524" layer="91"/>
 <label x="62" y="110" size="1.778" layer="95" rot="R90"/>
+</segment>
+<segment>
+<pinref part="R19" gate="G$1" pin="2"/>
+<wire x1="-77" y1="-88.08" x2="-77" y2="-94" width="0.1524" layer="91"/>
+<pinref part="R20" gate="G$1" pin="2"/>
+<wire x1="-77" y1="-94" x2="-81.92" y2="-94" width="0.1524" layer="91"/>
+<wire x1="-99" y1="-88" x2="-77" y2="-88" width="0.1524" layer="91"/>
+<wire x1="-77" y1="-88" x2="-77" y2="-88.08" width="0.1524" layer="91"/>
+<junction x="-77" y="-88.08"/>
+<label x="-106" y="-88" size="1.778" layer="95"/>
 </segment>
 </net>
@@
 <wire x1="39" y1="-187" x2="15" y2="-187" width="0.1524" layer="91"/>
 </segment>
+<segment>
+<pinref part="R18" gate="G$1" pin="2"/>
+<wire x1="-96.08" y1="-64" x2="-99" y2="-64" width="0.1524" layer="91"/>
+<label x="-104" y="-64" size="1.778" layer="95"/>
+</segment>
+<segment>
+<pinref part="J12" gate="G$1" pin="1"/>
+<wire x1="-72" y1="-66" x2="-99" y2="-66" width="0.1524" layer="91"/>
+<label x="-104" y="-66" size="1.778" layer="95"/>
+</segment>
 </net>
 <net name="N$2" class="0">
@@
 </segment>
 </net>
+<net name="N$11" class="0">
+<segment>
+<pinref part="R18" gate="G$1" pin="1"/>
+<pinref part="MOSFET1" gate="G$1" pin="D"/>
+<wire x1="-85.92" y1="-64" x2="-83.46" y2="-64" width="0.1524" layer="91"/>
+<wire x1="-83.46" y1="-64" x2="-83.46" y2="-69.38" width="0.1524" layer="91"/>
+<pinref part="J12" gate="G$1" pin="3"/>
+<wire x1="-72" y1="-71.08" x2="-83.46" y2="-71.08" width="0.1524" layer="91"/>
+<wire x1="-83.46" y1="-71.08" x2="-83.46" y2="-69.38" width="0.1524" layer="91"/>
+<junction x="-83.46" y="-69.38"/>
+</segment>
+</net>
+<net name="N$13" class="0">
+<segment>
+<pinref part="J12" gate="G$1" pin="2"/>
+<pinref part="R19" gate="G$1" pin="1"/>
+<wire x1="-72" y1="-68.54" x2="-77" y2="-68.54" width="0.1524" layer="91"/>
+<wire x1="-77" y1="-68.54" x2="-77" y2="-77.92" width="0.1524" layer="91"/>
+</segment>
+</net>

Commit message: .sch、.brd共に完成
Parts:
- added J16: B2B-XH-A_LF__SN_, B2B-XH-A_LF__SN_:B2B-XH-A_LF__SN_
Connections:
- net +3.3V: now also J16.1
- net CAN_TX: no longer R5.2
- net LED_TX: now also R5.2
- net MSW6: now also J16.2
Changed lines of the file:
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@@
 <setting verticaltext="up"/>
 </settings>
-<grid distance="1" unitdist="mm" unit="mm" style="lines" multiple="1" display="yes" altdistance="0.01" altunitdist="inch" altunit="mm"/>
+<grid distance="1" unitdist="mm" unit="mm" style="lines" multiple="1" display="yes" altdistance="0.25" altunitdist="mm" altunit="mm"/>
 <layers>
 <layer number="1" name="Top" color="4" fill="1" visible="no" active="no"/>
@@
 <part name="R19" library="rcl" library_urn="urn:adsk.eagle:library:334" deviceset="R-US_" device="R0603" package3d_urn="urn:adsk.eagle:package:23555/3" value="1k"/>
 <part name="R20" library="rcl" library_urn="urn:adsk.eagle:library:334" deviceset="R-US_" device="R0603" package3d_urn="urn:adsk.eagle:package:23555/3" value="2k"/>
+<part name="J16" library="B2B-XH-A_LF__SN_" deviceset="B2B-XH-A_LF__SN_" device=""/>
 </parts>
 <sheets>
@@
 <attribute name="NAME" x="-90.81" y="-92.5014" size="1.778" layer="95"/>
 <attribute name="VALUE" x="-90.81" y="-97.302" size="1.778" layer="96"/>
+</instance>
+<instance part="J16" gate="G$1" x="144" y="-184" smashed="yes">
+<attribute name="NAME" x="160.51" y="-176.38" size="1.778" layer="95" align="center-left"/>
+<attribute name="VALUE" x="160.51" y="-178.92" size="1.778" layer="96" align="center-left"/>
 </instance>
 </instances>
@@
 <segment>
 <pinref part="IC1" gate="G$1" pin="VDD_1"/>
-<wire x1="39" y1="66" x2="17.08" y2="66" width="0.1524" layer="91"/>
+<wire x1="39" y1="66" x2="6" y2="66" width="0.1524" layer="91"/>
+<label x="-1" y="65" size="1.778" layer="95"/>
 <pinref part="C1" gate="G$1" pin="2"/>
-<wire x1="17" y1="66" x2="6" y2="66" width="0.1524" layer="91"/>
 <wire x1="17.08" y1="70" x2="17.08" y2="66" width="0.1524" layer="91"/>
-<wire x1="17.08" y1="66" x2="17" y2="66" width="0.1524" layer="91"/>
-<junction x="17" y="66"/>
-<label x="-1" y="65" size="1.778" layer="95"/>
+<wire x1="17.08" y1="66" x2="39" y2="66" width="0.1524" layer="91"/>
+<junction x="39" y="66"/>
 </segment>
 <segment>
@@
 <pinref part="R4" gate="G$1" pin="2"/>
 <wire x1="-14" y1="106.08" x2="-14" y2="109" width="0.1524" layer="91"/>
+<label x="-14" y="110" size="1.778" layer="95" rot="R90"/>
 </segment>
 <segment>
@@
 <wire x1="-86" y1="-181" x2="-99" y2="-181" width="0.1524" layer="91"/>
 <label x="-106" y="-181" size="1.778" layer="95"/>
+</segment>
+<segment>
+<pinref part="J16" gate="G$1" pin="1"/>
+<wire x1="144" y1="-184" x2="139" y2="-184" width="0.1524" layer="91"/>
+<label x="132" y="-184" size="1.778" layer="95"/>
 </segment>
 </net>
@@
 <wire x1="39" y1="-110.54" x2="15" y2="-110.54" width="0.1524" layer="91"/>
 <wire x1="15" y1="-110.54" x2="15" y2="-111" width="0.1524" layer="91"/>
+<label x="9" y="-111" size="1.778" layer="95"/>
 </segment>
 <segment>
 <pinref part="R9" gate="G$1" pin="1"/>
 <wire x1="15.92" y1="-116" x2="15" y2="-116" width="0.1524" layer="91"/>
+<label x="9" y="-116" size="1.778" layer="95"/>
 </segment>
 <segment>
@@
 <wire x1="39" y1="-130.54" x2="15" y2="-130.54" width="0.1524" layer="91"/>
 <wire x1="15" y1="-130.54" x2="15" y2="-130" width="0.1524" layer="91"/>
+<label x="9" y="-131" size="1.778" layer="95"/>
 </segment>
 <segment>
 <pinref part="R11" gate="G$1" pin="1"/>
 <wire x1="15.92" y1="-136" x2="15" y2="-136" width="0.1524" layer="91"/>
+<label x="9" y="-137" size="1.778" layer="95"/>
 </segment>
 <segment>
@@
 <wire x1="39" y1="-150.54" x2="15" y2="-150.54" width="0.1524" layer="91"/>
 <wire x1="15" y1="-150.54" x2="15" y2="-151" width="0.1524" layer="91"/>
+<label x="9" y="-151" size="1.778" layer="95"/>
 </segment>
 <segment>
 <pinref part="R13" gate="G$1" pin="1"/>
 <wire x1="15.92" y1="-155" x2="15" y2="-155" width="0.1524" layer="91"/>
+<label x="9" y="-156" size="1.778" layer="95"/>
 </segment>
 <segment>
@@
 <wire x1="39" y1="-169.54" x2="15" y2="-169.54" width="0.1524" layer="91"/>
 <wire x1="15" y1="-169.54" x2="15" y2="-169" width="0.1524" layer="91"/>
+<label x="9" y="-170" size="1.778" layer="95"/>
 </segment>
 <segment>
 <pinref part="R15" gate="G$1" pin="1"/>
 <wire x1="15.92" y1="-175" x2="15" y2="-175" width="0.1524" layer="91"/>
+<label x="9" y="-176" size="1.778" layer="95"/>
 </segment>
 <segment>
@@
 <wire x1="39" y1="-189.54" x2="15" y2="-189.54" width="0.1524" layer="91"/>
 <wire x1="15" y1="-189.54" x2="15" y2="-189" width="0.1524" layer="91"/>
+<label x="9" y="-190" size="1.778" layer="95"/>
 </segment>
 <segment>
 <pinref part="R17" gate="G$1" pin="1"/>
 <wire x1="15.92" y1="-195" x2="15" y2="-195" width="0.1524" layer="91"/>
+<label x="9" y="-195" size="1.778" layer="95"/>
 </segment>
 <segment>
@@
 <wire x1="27.92" y1="-195" x2="26.08" y2="-195" width="0.1524" layer="91"/>
 <junction x="27.92" y="-192"/>
+<label x="10" y="-192" size="1.778" layer="95"/>
 </segment>
 </net>
@@
 <wire x1="27.92" y1="-175" x2="26.08" y2="-175" width="0.1524" layer="91"/>
 <junction x="27.92" y="-172"/>
+<label x="9" y="-173" size="1.778" layer="95"/>
 </segment>
 </net>
@@
 </segment>
 </net>
-<net name="LED_TX" class="0">
-<segment>
-<pinref part="IC1" gate="G$1" pin="PB3"/>
-<wire x1="64.4" y1="83.78" x2="64.4" y2="109" width="0.1524" layer="91"/>
-<wire x1="64.4" y1="109" x2="64" y2="109" width="0.1524" layer="91"/>
-<label x="65" y="110" size="1.778" layer="95" rot="R90"/>
-</segment>
-</net>
 <net name="VCP_RX" class="0">
 <segment>
@@
 <label x="61" y="-40" size="1.778" layer="95"/>
 </segment>
-<segment>
-<pinref part="R5" gate="G$1" pin="2"/>
-<wire x1="-3" y1="106.08" x2="-3" y2="109" width="0.1524" layer="91"/>
-</segment>
 </net>
 <net name="CAN_RX" class="0">
@@
 <wire x1="144" y1="-103" x2="139" y2="-103" width="0.1524" layer="91"/>
 <label x="131" y="-104" size="1.778" layer="95"/>
-</segment>
-</net>
-<net name="MSW6" class="0">
-<segment>
-<pinref part="IC1" gate="G$1" pin="PA7"/>
-<wire x1="59.32" y1="30.44" x2="59.32" y2="8" width="0.1524" layer="91"/>
-<wire x1="59.32" y1="8" x2="60" y2="8" width="0.1524" layer="91"/>
-<label x="60" y="0" size="1.778" layer="95" rot="R90"/>
 </segment>
 </net>
@@
 <wire x1="27.92" y1="-116" x2="26.08" y2="-116" width="0.1524" layer="91"/>
 <junction x="27.92" y="-113"/>
+<label x="10" y="-113" size="1.778" layer="95"/>
 </segment>
 </net>
@@
 <wire x1="27.92" y1="-136" x2="26.08" y2="-136" width="0.1524" layer="91"/>
 <junction x="27.92" y="-133"/>
+<label x="9" y="-134" size="1.778" layer="95"/>
 </segment>
 </net>
@@
 <wire x1="27.92" y1="-155" x2="26.08" y2="-155" width="0.1524" layer="91"/>
 <junction x="27.92" y="-153"/>
+<label x="10" y="-153" size="1.778" layer="95"/>
 </segment>
 </net>
@@
 <pinref part="J7" gate="G$1" pin="1"/>
 <wire x1="39" y1="-108" x2="15" y2="-108" width="0.1524" layer="91"/>
+<label x="10" y="-108" size="1.778" layer="95"/>
 </segment>
 <segment>
 <pinref part="J8" gate="G$1" pin="1"/>
 <wire x1="39" y1="-128" x2="15" y2="-128" width="0.1524" layer="91"/>
+<label x="9" y="-128" size="1.778" layer="95"/>
 </segment>
 <segment>
 <pinref part="J9" gate="G$1" pin="1"/>
 <wire x1="39" y1="-148" x2="15" y2="-148" width="0.1524" layer="91"/>
+<label x="9" y="-148" size="1.778" layer="95"/>
 </segment>
 <segment>
 <pinref part="J10" gate="G$1" pin="1"/>
 <wire x1="39" y1="-167" x2="15" y2="-167" width="0.1524" layer="91"/>
+<label x="10" y="-167" size="1.778" layer="95"/>
 </segment>
 <segment>
 <pinref part="J11" gate="G$1" pin="1"/>
 <wire x1="39" y1="-187" x2="15" y2="-187" width="0.1524" layer="91"/>
+<label x="10" y="-188" size="1.778" layer="95"/>
 </segment>
 <segment>
@@
 </segment>
 </net>
+<net name="LED_TX" class="0">
+<segment>
+<pinref part="IC1" gate="G$1" pin="PB3"/>
+<wire x1="64.4" y1="83.78" x2="64.4" y2="109" width="0.1524" layer="91"/>
+<wire x1="64.4" y1="109" x2="64" y2="109" width="0.1524" layer="91"/>
+<label x="65" y="110" size="1.778" layer="95" rot="R90"/>
+</segment>
+<segment>
+<pinref part="R5" gate="G$1" pin="2"/>
+<wire x1="-3" y1="106.08" x2="-3" y2="109" width="0.1524" layer="91"/>
+<label x="-3" y="110" size="1.778" layer="95" rot="R90"/>
+</segment>
+</net>
+<net name="MSW6" class="0">
+<segment>
+<pinref part="IC1" gate="G$1" pin="PA7"/>
+<wire x1="59.32" y1="30.44" x2="59.32" y2="8" width="0.1524" layer="91"/>
+<wire x1="59.32" y1="8" x2="59" y2="8" width="0.1524" layer="91"/>
+<label x="60" y="0" size="1.778" layer="95" rot="R90"/>
+</segment>
+<segment>
+<pinref part="J16" gate="G$1" pin="2"/>
+<wire x1="144" y1="-186.54" x2="139" y2="-186.54" width="0.1524" layer="91"/>
+<wire x1="139" y1="-186.54" x2="139" y2="-187" width="0.1524" layer="91"/>
+<label x="131" y="-187" size="1.778" layer="95"/>
+</segment>
+</net>
